Commit message: update section08

File: src/my_robot_description/urdf/common_properties.xacro (robot description, xacro)
@@ -7,11 +7,15 @@
         <color rgba="0.5 0.5 0.5 1" />
     </material>
+    <material name="orange">
+        <color rgba="1 0.5 0 1" />
+    </material>
+    <material name="yellow">
+        <color rgba="1 1 0 1" />
+    </material>
     <xacro:macro name="box_inertia" params="m l w h xyz rpy">
         <inertial>
             <origin xyz="${xyz}" rpy="${rpy}" />
             <mass value="${m}" />
-            <inertia ixx="${(m / 12) * (h**2 + l**2)}" ixy="0" ixz="0"
-                     iyy="${(m / 12) * (w**2 + l**2)}" iyz="0"
-                     izz="${(m / 12) * (w**2 + h**2)}" />
+            <inertia ixx="${(m / 12) * (h**2 + l**2)}" ixy="0" ixz="0" iyy="${(m / 12) * (w**2 + l**2)}" iyz="0" izz="${(m / 12) * (w**2 + h**2)}" />
         </inertial>
     </xacro:macro>
@@ -20,7 +24,5 @@
             <origin xyz="${xyz}" rpy="${rpy}" />
             <mass value="${m}" />
-            <inertia ixx="${(m / 12) * (3 * r**2 + h**2)}" ixy="0" ixz="0"
-                     iyy="${(m / 12) * (3 * r**2 + h**2)}" iyz="0"
-                     izz="${(m / 2) * (r**2)}" />
+            <inertia ixx="${(m / 12) * (3 * r**2 + h**2)}" ixy="0" ixz="0" iyy="${(m / 12) * (3 * r**2 + h**2)}" iyz="0" izz="${(m / 2) * (r**2)}" />
         </inertial>
     </xacro:macro>
@@ -29,7 +31,5 @@
             <origin xyz="${xyz}" rpy="${rpy}" />
             <mass value="${m}" />
-            <inertia ixx="${(2 * m / 5) * (r**2)}" ixy="0" ixz="0"
-                     iyy="${(2 * m / 5) * (r**2)}" iyz="0"
-                     izz="${(2 * m / 5) * (r**2)}" />
+            <inertia ixx="${(2 * m / 5) * (r**2)}" ixy="0" ixz="0" iyy="${(2 * m / 5) * (r**2)}" iyz="0" izz="${(2 * m / 5) * (r**2)}" />
         </inertial>
     </xacro:macro>
