Commit message: add collision tags

File: src/my_robot_description/urdf/arm.xacro (robot description, xacro)
@@ -16,4 +16,10 @@
             <material name="orange" />
         </visual>
+        <collision>
+            <geometry>
+                <box size="${arm_base_length} ${arm_base_width} ${arm_base_height}" />
+            </geometry>
+            <origin xyz="0 0 ${arm_base_height / 2.0}" rpy="0 0 0" />
+        </collision>
     </link>
     <link name="forearm_link">
@@ -25,4 +31,10 @@
             <material name="yellow" />
         </visual>
+        <collision>
+            <geometry>
+                <cylinder radius="${forearm_radius}" length="${forearm_length}"/>
+            </geometry>
+            <origin xyz="0 0 ${forearm_length / 2.0}" rpy="0 0 0" />
+        </collision>
     </link>
     <link name="hand_link">
@@ -34,4 +46,10 @@
             <material name="orange" />
         </visual>
+        <collision>
+            <geometry>
+                <cylinder radius="${hand_radius}" length="${hand_length}"/>
+            </geometry>
+            <origin xyz="0 0 ${hand_length / 2.0}" rpy="0 0 0" />
+        </collision>
     </link>
     <joint name="arm_base_forearm_joint" type="revolute">

Commit message: update for robotic arm

File: src/my_robot_description/urdf/arm.xacro (robot description, xacro)
@@ -22,4 +22,5 @@
             <origin xyz="0 0 ${arm_base_height / 2.0}" rpy="0 0 0" />
         </collision>
+        <xacro:box_inertia m="0.5" l="${2.0 * arm_base_length}" w="${2.0 * arm_base_width}" h="${2.0 * arm_base_height}" xyz="0 0 ${arm_base_height / 2.0}" rpy="0 0 0" />
     </link>
     <link name="forearm_link">
@@ -37,4 +38,5 @@
             <origin xyz="0 0 ${forearm_length / 2.0}" rpy="0 0 0" />
         </collision>
+        <xacro:cylinder_inertia m="0.3" r="${forearm_radius}" h="${forearm_length}" xyz="0 0 ${forearm_length / 2.0}" rpy="0 0 0" />
     </link>
     <link name="hand_link">
@@ -52,4 +54,5 @@
             <origin xyz="0 0 ${hand_length / 2.0}" rpy="0 0 0" />
         </collision>
+        <xacro:cylinder_inertia m="0.3" r="${hand_radius}" h="${hand_length}" xyz="0 0 ${hand_length / 2.0}" rpy="0 0 0" />
     </link>
     <joint name="arm_base_forearm_joint" type="revolute">
@@ -59,4 +62,5 @@
         <axis xyz="0 1 0" />
         <limit lower="0" upper="${pi/2}" effort="100" velocity="100" />
+        <dynamics friction="0.05" damping="0.1" />
     </joint>
     <joint name="forearm_hand_joint" type="revolute">
@@ -66,4 +70,5 @@
         <axis xyz="0 1 0" />
         <limit lower="0" upper="${pi/2}" effort="100" velocity="100" />
+        <dynamics friction="0.05" damping="0.1" />
     </joint>
 </robot>

File: src/my_robot_description/urdf/my_robot.urdf.xacro (robot description, xacro)
@@ -6,3 +6,10 @@
     <xacro:include filename="camera.xacro" />
     <xacro:include filename="camera_gazebo.xacro" />
+    <xacro:include filename="arm.xacro" />
+    <xacro:include filename="arm_gazebo.xacro" />
+    <joint name="mobile_base_arm_joint" type="fixed">
+        <parent link="base_footprint" />
+        <child link="arm_base_link" />
+        <origin xyz="${base_length / 4.0} 0 ${base_height + wheel_radius}" rpy="0 0 0" />
+    </joint>
 </robot>

File: src/my_robot_description/urdf/standalone_arm.urdf.xacro (robot description, xacro)
@@ -3,3 +3,4 @@
     <xacro:include filename="common_properties.xacro" />
     <xacro:include filename="arm.xacro" />
+    <xacro:include filename="arm_gazebo.xacro" />
 </robot>
